File: connectors.kicad_sch (KiCad schematic)
At the start: 7 parts, among them J1 USB_A

Commit message: schem: export revision info to all sheets
Other:
- title: (none) -> RepRapDiscount.com Smart Controller
Changed lines of the file:
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@@
 (kicad_sch (version 20230121) (generator eeschema)
-  (paper "A4")
+  (paper "A")
+  (title_block
+    (title "RepRapDiscount.com Smart Controller")
+    (date "${DATE}")
+    (rev "${TAG} (${HASH})")
+  )
   (junction (at 189.23 93.98) (diameter 0) (color 0 0 0 0)
   )
